Commit message: diablo balance is work

File: diablo_train-main/resources/robots/diablo/urdf/diablo_asm.urdf (robot description, URDF)
Before this commit: robot diablo_ASM, 7 links, 6 joints
Links:
- removed link left_fake_shank_link
- removed link left_fake_thigh_link
- removed link right_fake_shank_link
- removed link right_fake_thigh_link
- added link left_shank_link, mass 0.071103; collision mesh filename=../meshes/left_leg3.STL scale=1 1 1; visual mesh filename=../meshes/left_leg3.STL scale=1 1 1
- added link left_thigh_link, mass 2.5; collision mesh filename=../meshes/left_motor.STL scale=1 1 1; visual mesh filename=../meshes/left_motor.STL scale=1 1 1
- added link right_shank_link, mass 0.071103; collision mesh filename=../meshes/right_leg3.STL scale=1 1 1; visual mesh filename=../meshes/right_leg3.STL scale=1 1 1
- added link right_thigh_link, mass 2.5; collision mesh filename=../meshes/right_motor.STL scale=1 1 1; visual mesh filename=../meshes/right_motor.STL scale=1 1 1
Joints:
- removed joint left_fake_hip_joint
- removed joint left_fake_knee_joint
- removed joint right_fake_hip_joint
- removed joint right_fake_knee_joint
- added joint left_hip_joint: type revolute, parent diablo_base_link, child left_thigh_link, origin xyz=0 0.18755 0 rpy=1.5708 0.13433 -3.1416, axis 0 0 1, limit lower=-1.57 upper=1.57 effort=27 velocity=26
- added joint left_knee_joint: type revolute, parent left_thigh_link, child left_shank_link, origin xyz=0.14 0 0 rpy=0 0 -2.8729, axis 0 0 1, limit lower=-1.57 upper=1.57 effort=27 velocity=26
- added joint right_hip_joint: type revolute, parent diablo_base_link, child right_thigh_link, origin xyz=0 -0.18755 0 rpy=1.5708 0.13433 3.1416, axis 0 0 1, limit lower=-1.57 upper=1.57 effort=27 velocity=26
- added joint right_knee_joint: type revolute, parent right_thigh_link, child right_shank_link, origin xyz=0.14 0 0 rpy=0 0 -2.8729, axis 0 0 1, limit lower=-1.57 upper=1.57 effort=27 velocity=26
- joint left_wheel_joint: parent left_fake_shank_link -> left_shank_link
- joint right_wheel_joint: parent right_fake_shank_link -> right_shank_link
